File: fan7385_breakout.sch (EAGLE design)
At the start: 15 parts

Commit message: added some caps
Parts:
- added CVDD1, CVDD2: 0.1uF 25V, microbuilder:CAP_CERAMIC0805
Connections:
- net GND: now also CVDD1.P$1, CVDD2.P$1
- net VDD: now also CVDD1.P$2, CVDD2.P$2
Changed lines of the file:
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@@
 <part name="JP3" library="SparkFun-Connectors" deviceset="M03" device="PTH"/>
 <part name="JP4" library="SparkFun-Connectors" deviceset="M03" device="PTH"/>
+<part name="CVDD1" library="microbuilder" deviceset="CAP_CERAMIC" device="0805" value="0.1uF 25V"/>
+<part name="CVDD2" library="microbuilder" deviceset="CAP_CERAMIC" device="0805" value="0.1uF 25V"/>
 </parts>
 <sheets>
@@
 <instance part="JP3" gate="G$1" x="137.16" y="55.88"/>
 <instance part="JP4" gate="G$1" x="137.16" y="38.1"/>
+<instance part="CVDD1" gate="G$1" x="53.34" y="2.54" smashed="yes" rot="R270">
+<attribute name="NAME" x="53.34" y="0" size="1.27" layer="95" font="vector"/>
+<attribute name="VALUE" x="58.42" y="5.08" size="1.27" layer="96" font="vector" rot="R180"/>
+</instance>
+<instance part="CVDD2" gate="G$1" x="53.34" y="-10.16" smashed="yes" rot="R270">
+<attribute name="NAME" x="53.34" y="-12.7" size="1.27" layer="95" font="vector"/>
+<attribute name="VALUE" x="58.42" y="-7.62" size="1.27" layer="96" font="vector" rot="R180"/>
+</instance>
 </instances>
 <busses>
@@
 <pinref part="JP1" gate="G$1" pin="1"/>
 <junction x="0" y="45.72"/>
+</segment>
+<segment>
+<pinref part="CVDD1" gate="G$1" pin="P$1"/>
+<wire x1="58.42" y1="2.54" x2="60.96" y2="2.54" width="0.1524" layer="91"/>
+<label x="60.96" y="2.54" size="1.778" layer="95"/>
+</segment>
+<segment>
+<pinref part="CVDD2" gate="G$1" pin="P$1"/>
+<wire x1="58.42" y1="-10.16" x2="60.96" y2="-10.16" width="0.1524" layer="91"/>
+<label x="60.96" y="-10.16" size="1.778" layer="95"/>
 </segment>
 </net>
@@
 <junction x="0" y="55.88"/>
 </segment>
+<segment>
+<pinref part="CVDD1" gate="G$1" pin="P$2"/>
+<wire x1="50.8" y1="2.54" x2="48.26" y2="2.54" width="0.1524" layer="91"/>
+<label x="43.18" y="2.54" size="1.778" layer="95"/>
+</segment>
+<segment>
+<pinref part="CVDD2" gate="G$1" pin="P$2"/>
+<wire x1="50.8" y1="-10.16" x2="48.26" y2="-10.16" width="0.1524" layer="91"/>
+<label x="43.18" y="-10.16" size="1.778" layer="95"/>
+</segment>
 </net>

Commit message: removed a cap to help with routing
Parts:
- removed CVDD2: 0.1uF 25V, microbuilder:CAP_CERAMIC0805
Connections:
- net GND: no longer CVDD2.P$1
- net VDD: no longer CVDD2.P$2
Changed lines of the file:
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@@
 <part name="JP4" library="SparkFun-Connectors" deviceset="M03" device="PTH"/>
 <part name="CVDD1" library="microbuilder" deviceset="CAP_CERAMIC" device="0805" value="0.1uF 25V"/>
-<part name="CVDD2" library="microbuilder" deviceset="CAP_CERAMIC" device="0805" value="0.1uF 25V"/>
 </parts>
 <sheets>
@@
 <attribute name="VALUE" x="58.42" y="5.08" size="1.27" layer="96" font="vector" rot="R180"/>
 </instance>
-<instance part="CVDD2" gate="G$1" x="53.34" y="-10.16" smashed="yes" rot="R270">
-<attribute name="NAME" x="53.34" y="-12.7" size="1.27" layer="95" font="vector"/>
-<attribute name="VALUE" x="58.42" y="-7.62" size="1.27" layer="96" font="vector" rot="R180"/>
-</instance>
 </instances>
 <busses>
@@
 <wire x1="58.42" y1="2.54" x2="60.96" y2="2.54" width="0.1524" layer="91"/>
 <label x="60.96" y="2.54" size="1.778" layer="95"/>
-</segment>
-<segment>
-<pinref part="CVDD2" gate="G$1" pin="P$1"/>
-<wire x1="58.42" y1="-10.16" x2="60.96" y2="-10.16" width="0.1524" layer="91"/>
-<label x="60.96" y="-10.16" size="1.778" layer="95"/>
 </segment>
 </net>
@@
 <label x="43.18" y="2.54" size="1.778" layer="95"/>
 </segment>
-<segment>
-<pinref part="CVDD2" gate="G$1" pin="P$2"/>
-<wire x1="50.8" y1="-10.16" x2="48.26" y2="-10.16" width="0.1524" layer="91"/>
-<label x="43.18" y="-10.16" size="1.778" layer="95"/>
-</segment>
 </net>

Commit message: routed
Parts:
- added CVDD2: 0.1uF 25V, microbuilder:CAP_CERAMIC0805
Connections:
- net GND: now also CVDD2.P$1
- net VDD: now also CVDD2.P$2
Changed lines of the file:
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@@
 <part name="JP4" library="SparkFun-Connectors" deviceset="M03" device="PTH"/>
 <part name="CVDD1" library="microbuilder" deviceset="CAP_CERAMIC" device="0805" value="0.1uF 25V"/>
+<part name="CVDD2" library="microbuilder" deviceset="CAP_CERAMIC" device="0805" value="0.1uF 25V"/>
 </parts>
 <sheets>
@@
 <attribute name="VALUE" x="58.42" y="5.08" size="1.27" layer="96" font="vector" rot="R180"/>
 </instance>
+<instance part="CVDD2" gate="G$1" x="53.34" y="-7.62" smashed="yes" rot="R270">
+<attribute name="NAME" x="53.34" y="-10.16" size="1.27" layer="95" font="vector"/>
+<attribute name="VALUE" x="58.42" y="-5.08" size="1.27" layer="96" font="vector" rot="R180"/>
+</instance>
 </instances>
 <busses>
@@
 <wire x1="58.42" y1="2.54" x2="60.96" y2="2.54" width="0.1524" layer="91"/>
 <label x="60.96" y="2.54" size="1.778" layer="95"/>
+</segment>
+<segment>
+<pinref part="CVDD2" gate="G$1" pin="P$1"/>
+<wire x1="58.42" y1="-7.62" x2="60.96" y2="-7.62" width="0.1524" layer="91"/>
+<label x="60.96" y="-7.62" size="1.778" layer="95"/>
 </segment>
 </net>
@@
 <label x="43.18" y="2.54" size="1.778" layer="95"/>
 </segment>
+<segment>
+<pinref part="CVDD2" gate="G$1" pin="P$2"/>
+<wire x1="50.8" y1="-7.62" x2="48.26" y2="-7.62" width="0.1524" layer="91"/>
+<label x="43.18" y="-7.62" size="1.778" layer="95"/>
+</segment>
 </net>

Commit message: UAAH! mixed source and drain for the cboot return...
Connections:
- net D1: no longer SJ3.2
- net D2: no longer SJ4.2
- net S1: now also SJ3.2
- net S2: now also SJ4.2
Changed lines of the file:
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@@
 <junction x="144.78" y="35.56"/>
+</segment>
+<segment>
+<pinref part="SJ3" gate="1" pin="2"/>
+<wire x1="111.76" y1="22.86" x2="114.3" y2="22.86" width="0.1524" layer="91"/>
+<label x="114.3" y="22.86" size="1.778" layer="95"/>
 </segment>
 </net>
@@
 <pinref part="JP3" gate="G$1" pin="1"/>
 <junction x="144.78" y="53.34"/>
+</segment>
+<segment>
+<pinref part="SJ4" gate="1" pin="2"/>
+<wire x1="111.76" y1="15.24" x2="114.3" y2="15.24" width="0.1524" layer="91"/>
+<label x="114.3" y="15.24" size="1.778" layer="95"/>
 </segment>
 </net>
@@
 <junction x="144.78" y="58.42"/>
 </segment>
-<segment>
-<pinref part="SJ4" gate="1" pin="2"/>
-<wire x1="111.76" y1="15.24" x2="114.3" y2="15.24" width="0.1524" layer="91"/>
-<label x="114.3" y="15.24" size="1.778" layer="95"/>
-</segment>
 </net>
 <net name="D1" class="2">
@@
 <junction x="144.78" y="40.64"/>
 </segment>
-<segment>
-<pinref part="SJ3" gate="1" pin="2"/>
-<wire x1="111.76" y1="22.86" x2="114.3" y2="22.86" width="0.1524" layer="91"/>
-<label x="114.3" y="22.86" size="1.778" layer="95"/>
-</segment>
 </net>

Commit message: these should be connected to drain as well, but now we have a problem with routing
Connections:
- net D1: now also SJ2.2
- net D2: now also SJ1.2
- net S1: no longer SJ2.2
- net S2: no longer SJ1.2
Changed lines of the file:
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@@
-</segment>
-<segment>
-<pinref part="SJ2" gate="1" pin="2"/>
-<wire x1="111.76" y1="58.42" x2="114.3" y2="58.42" width="0.1524" layer="91"/>
-<label x="114.3" y="58.42" size="1.778" layer="95"/>
 </segment>
 <segment>
@@
 <wire x1="86.36" y1="35.56" x2="86.36" y2="22.86" width="0.1524" layer="91"/>
 <label x="86.36" y="20.32" size="1.778" layer="95"/>
-</segment>
-<segment>
-<pinref part="SJ1" gate="1" pin="2"/>
-<wire x1="111.76" y1="50.8" x2="114.3" y2="50.8" width="0.1524" layer="91"/>
-<label x="114.3" y="50.8" size="1.778" layer="95"/>
 </segment>
 <segment>
@@
 <junction x="144.78" y="58.42"/>
 </segment>
+<segment>
+<pinref part="SJ1" gate="1" pin="2"/>
+<wire x1="111.76" y1="50.8" x2="114.3" y2="50.8" width="0.1524" layer="91"/>
+<label x="114.3" y="50.8" size="1.778" layer="95"/>
+</segment>
 </net>
 <net name="D1" class="2">
@@
 <junction x="144.78" y="40.64"/>
 </segment>
+<segment>
+<pinref part="SJ2" gate="1" pin="2"/>
+<wire x1="111.76" y1="58.42" x2="114.3" y2="58.42" width="0.1524" layer="91"/>
+<label x="114.3" y="58.42" size="1.778" layer="95"/>
+</segment>
 </net>
